Commit message: Updated Gazebo Workshop

File: tutorials/workshop_examples/urdf/diff_wheeled_robot.xacro (robot description, xacro)
@@ -1,20 +1,6 @@
 <?xml version="1.0"?>
 <robot name="differential_wheeled_robot" xmlns:xacro="http://www.ros.org/wiki/xacro">
-  <xacro:include filename="$(find diff_wheeled_robot_description)/urdf/wheel.urdf.xacro" />
-  <xacro:include filename="$(find diff_wheeled_robot_description)/urdf/sonar_model.xacro"/>
-<!-- Defining the colors used in this robot -->
-  <material name="Black">
-    <color rgba="0.0 0.0 0.0 1.0"/>
-  </material>
-  <material name="Red">
-    <color rgba="0.8 0.0 0.0 1.0"/>
-  </material>
-  <material name="White">
-    <color rgba="1.0 1.0 1.0 1.0"/>
-  </material>
-  <material name="Blue">
-    <color rgba="0.0 0.0 0.8 1.0"/>
-  </material>
-  <!-- PROPERTY LIST -->
+<xacro:include filename="$(find diff_wheeled_robot_description)/urdf/sonar_model.xacro"/>
+ <!-- PROPERTY LIST -->
   <!--All units in m-kg-s-radians unit system -->
   <property name="M_PI" value="3.1415926535897931" />
@@ -36,6 +22,14 @@
   <property name="caster_b_radius" value="0.025" />
   <property name="caster_b_mass" value="0.5" /> <!-- in kg-->
-  <!-- Wheels -->
-  <property name="wheel_mass" value="2.5" /> --> <!-- in kg-->
+  <property name="wheel_radius" value="0.04" />
+  <property name="wheel_height" value="0.02" />
+  <property name="wheel_mass" value="2.5" /> <!-- in kg-->
+  <property name="base_x_origin_to_wheel_origin" value="0.25" />
+  <property name="base_y_origin_to_wheel_origin" value="0.3" />
+  <property name="base_z_origin_to_wheel_origin" value="0.0" />
+<!-- Wheels -->
+  <property name="wheel_radius" value="0.04" />
+  <property name="wheel_height" value="0.02" />
+  <property name="wheel_mass" value="2.5" /> <!-- in kg-->
   <property name="base_x_origin_to_wheel_origin" value="0.25" />
   <property name="base_y_origin_to_wheel_origin" value="0.3" />
@@ -43,10 +37,4 @@
   <!-- Hokuyo Laser scanner -->
   <property name="hokuyo_size" value="0.05" />
-  <!-- Macro for calculating inertia of cylinder -->
-  <macro name="cylinder_inertia" params="m r h">
-    <inertia  ixx="${m*(3*r*r+h*h)/12}" ixy = "0" ixz = "0"
-              iyy="${m*(3*r*r+h*h)/12}" iyz = "0"
-              izz="${m*r*r/2}" />
-  </macro>
   <!-- BASE-FOOTPRINT -->
   <!-- base_footprint is a fictitious link(frame) that is on the ground right below base_link origin -->
@@ -80,6 +68,7 @@
       <mass value="${base_mass}" />
       <origin xyz="0 0 0" />
-      <!--The 3x3 rotational inertia matrix. -->
-        <cylinder_inertia  m="${base_mass}" r="${base_radius}" h="${base_height}" />
+         <inertia ixx="0.001" ixy="0.0" ixz="0.0"
+                 iyy="0.001" iyz="0.0"
+                 izz="0.001" />
     </inertial>
     <visual>
@@ -88,5 +77,4 @@
           <cylinder length="${base_height}" radius="${base_radius}" />
       </geometry>
-      <material name="White" />
     </visual>
     <collision>
@@ -98,5 +86,4 @@
   </link>
   <gazebo reference="base_link">
-    <material>Gazebo/White</material>
     <turnGravityOff>false</turnGravityOff>
   </gazebo>
@@ -108,5 +95,4 @@
 	<sphere radius="${caster_f_radius}" />
       </geometry>
-      <material name="Black" />
     </visual>
       <collision>
@@ -139,5 +125,4 @@
 	<sphere radius="${caster_b_radius}" />
       </geometry>
-      <material name="Black" />
     </visual>
       <collision>
@@ -164,6 +149,98 @@
   </gazebo>
 <!-- Wheel Definitions -->
-  <wheel fb="front" lr="right" parent="base_link" translateX="0" translateY="0.5" flipY="1"/>
-  <wheel fb="front" lr="left" parent="base_link" translateX="0" translateY="-0.5" flipY="1"/>
+<!--right_wheel-->
+    <link name="front_right_wheel">
+      <visual>
+        <origin xyz="0 0 0" rpy="${1*M_PI/2} 0  0 " />
+        <geometry>
+          <cylinder length="${wheel_height}" radius="${wheel_radius}" />
+        </geometry>
+      </visual>
+      <collision>
+        <origin xyz="0 0 0" rpy="${1*M_PI/2} 0 0 " />
+        <geometry>
+          <cylinder length="${wheel_height}" radius="${wheel_radius}" />
+        </geometry>
+      </collision>
+      <inertial>
+        <mass value="${wheel_mass}" />
+        <origin xyz="0 0 0" />
+        <inertia ixx="0.001" ixy="0.0" ixz="0.0"
+                 iyy="0.001" iyz="0.0"
+                 izz="0.001" />
+      </inertial>
+    </link>
+    <joint name="front_right_wheel_joint" type="continuous">
+      <parent link="base_link"/>
+      <child link="front_right_wheel"/>
+      <origin xyz="${0 * base_x_origin_to_wheel_origin} ${0.5 * base_y_origin_to_wheel_origin} ${base_z_origin_to_wheel_origin}" rpy="0 0 0" />
+      <axis xyz="0 1 0" rpy="0  0" />
+      <limit effort="100" velocity="100"/>
+      <joint_properties damping="0.0" friction="0.0"/>
+    </joint>
+ <!-- Transmission is important to link the joints and the controller -->
+    <transmission name="front_right_wheel_joint_trans">
+      <type>transmission_interface/SimpleTransmission</type>
+      <joint name="front_right_wheel_joint" />
+      <actuator name="front_right_wheel_joint_motor">
+        <hardwareInterface>EffortJointInterface</hardwareInterface>
+        <mechanicalReduction>1</mechanicalReduction>
+      </actuator>
+    </transmission>
+   <gazebo reference="front_right_wheel">
+      <mu1 value="1.0"/>
+      <mu2 value="1.0"/>
+      <kp  value="10000000.0" />
+      <kd  value="1.0" />
+      <fdir1 value="1 0 0"/>
+      <turnGravityOff>false</turnGravityOff>
+    </gazebo>
+<!--left_wheel-->
+    <link name="front_left_wheel">
+      <visual>
+        <origin xyz="0 0 0" rpy="${1*M_PI/2} 0  0 " />
+        <geometry>
+          <cylinder length="${wheel_height}" radius="${wheel_radius}" />
+        </geometry>
+      </visual>
+      <collision>
+        <origin xyz="0 0 0" rpy="${1*M_PI/2} 0 0 " />
+        <geometry>
+          <cylinder length="${wheel_height}" radius="${wheel_radius}" />
+        </geometry>
+      </collision>
+      <inertial>
+        <mass value="${wheel_mass}" />
+        <origin xyz="0 0 0" />
+        <inertia ixx="0.001" ixy="0.0" ixz="0.0"
+                 iyy="0.001" iyz="0.0"
+                 izz="0.001" />
+      </inertial>
+    </link>
+    <joint name="front_left_wheel_joint" type="continuous">
+      <parent link="base_link"/>
+      <child link="front_left_wheel"/>
+      <origin xyz="${0 * base_x_origin_to_wheel_origin} ${-0.5 * base_y_origin_to_wheel_origin} ${base_z_origin_to_wheel_origin}" rpy="0 0 0" />
+      <axis xyz="0 1 0" rpy="0  0" />
+      <limit effort="100" velocity="100"/>
+      <joint_properties damping="0.0" friction="0.0"/>
+    </joint>
+ <!-- Transmission is important to link the joints and the controller -->
+    <transmission name="front_left_wheel_joint_trans">
+      <type>transmission_interface/SimpleTransmission</type>
+      <joint name="front_left_wheel_joint" />
+      <actuator name="front_left_wheel_joint_motor">
+        <hardwareInterface>EffortJointInterface</hardwareInterface>
+        <mechanicalReduction>1</mechanicalReduction>
+      </actuator>
+    </transmission>
+    <gazebo reference="front_left_wheel">
+      <mu1 value="1.0"/>
+      <mu2 value="1.0"/>
+      <kp  value="10000000.0" />
+      <kd  value="1.0" />
+      <fdir1 value="1 0 0"/>
+      <turnGravityOff>false</turnGravityOff>
+    </gazebo>
   <!-- SENSORS-->
   <sonar_sensor parent="base_link" name="differential_wheeled_robot" ros_topic="/distance" update_rate="10" min_range="0.2" max_range="1" field_of_view="25" ray_count="2" >

Commit message: Updated Gazebo Tutorial, addressed robins comments

File: tutorials/workshop_examples/urdf/diff_wheeled_robot.xacro (robot description, xacro)
@@ -40,11 +40,4 @@
   <!-- base_footprint is a fictitious link(frame) that is on the ground right below base_link origin -->
   <link name="base_footprint">
-    <inertial>
-      <mass value="0.0001" />
-      <origin xyz="0 0 0" />
-      <inertia ixx="0.0001" ixy="0.0" ixz="0.0"
-          iyy="0.0001" iyz="0.0"
-          izz="0.0001" />
-    </inertial>
     <visual>
         <origin xyz="0 0 0" rpy="0 0 0" />

File: tutorials/workshop_examples/urdf/myrobot.urdf (robot description, URDF)
Before this commit: robot myrobot, 3 links, 2 joints
Links:
- link arm: geometry collision cylinder length=0.25 radius=0.01; visual cylinder length=0.25 radius=0.01
- link base_footprint: mass 0.0001 -> None
